File: wifi_led_strip.sch (KiCad schematic (older format))
At the start: 14 parts, among them J1 Serial, J2 Power, J3 ESP01, J4 Leds, SW1 Flash, SW2 Reset, U1 TLV1117-33

Commit message: beginning of layout
Parts:
- J2: footprint (none) -> wifi_led_strip:USB_Micro-B_Wuerth-629105136821
Changed lines of the file:
@@
 F 0 "J2" H 4355 1917 50  0000 C CNN
 F 1 "Power" H 4355 1826 50  0000 C CNN
-F 2 "" H 4450 1400 50  0001 C CNN
+F 2 "wifi_led_strip:USB_Micro-B_Wuerth-629105136821" H 4450 1400 50  0001 C CNN
 F 3 "~" H 4450 1400 50  0001 C CNN
 	1    4300 1450

Commit message: finish routing
Connections:
- net labels added: ESP_TO_PC, FLASH, PC_TO_ESP
- net labels removed: CH_PD, CTSn, GPIO0, GPIO2, RTSn, RXD, TXD, VCC
Other:
- note added: "CH_PD"
- note added: "CTSn"
- note added: "GND"
- note added: "GPIO0"
- note added: "GPIO2"
- note added: "RESET"
- note added: "RTSn"
- note added: "RXD"
- note added: "TXD"
- note added: "VCC"
Changed lines of the file:
@@
 EESchema Schematic File Version 4
+LIBS:wifi_led_strip-cache
 EELAYER 26 0
 EELAYER END
@@
 	0    -1   1    0
 $EndComp
-Text Label 6200 4050 1    50   ~ 0
-GND
-Text Label 6300 4050 1    50   ~ 0
-GPIO2
-Text Label 6400 4050 1    50   ~ 0
-GPIO0
-Text Label 6500 4050 1    50   ~ 0
-RXD
-Text Label 6200 4550 3    50   ~ 0
-TXD
-Text Label 6300 4550 3    50   ~ 0
-CH_PD
-Text Label 6400 4550 3    50   ~ 0
-RESET
-Text Label 6500 4550 3    50   ~ 0
-VCC
 $Comp
 L Device:R R2
@@
 	3850 3950 4200 3950
 Connection ~ 4800 5500
-Text Label 3850 3950 0    50   ~ 0
-GND
-Text Label 3850 3850 0    50   ~ 0
-CTSn
-Text Label 3850 3750 0    50   ~ 0
-VCC
-Text Label 3850 3650 0    50   ~ 0
-TXD
-Text Label 3850 3550 0    50   ~ 0
-RXD
-Text Label 3850 3450 0    50   ~ 0
-RTSn
 NoConn ~ 3850 3850
 NoConn ~ 3850 3450
@@
 Wire Wire Line
 	5600 1150 5600 1250
+Text Notes 3850 3450 0    50   ~ 0
+RTSn
+Text Notes 3850 3550 0    50   ~ 0
+RXD
+Text Notes 3850 3650 0    50   ~ 0
+TXD
+Text Notes 3850 3750 0    50   ~ 0
+VCC
+Text Notes 3850 3850 0    50   ~ 0
+CTSn
+Text Notes 3850 3950 0    50   ~ 0
+GND
+Text Notes 6200 4050 1    50   ~ 0
+GND
+Text Notes 6300 4050 1    50   ~ 0
+GPIO2
+Text Notes 6400 4050 1    50   ~ 0
+GPIO0
+Text Notes 6500 4050 1    50   ~ 0
+RXD
+Text Notes 6200 4550 3    50   ~ 0
+TXD
+Text Notes 6300 4550 3    50   ~ 0
+CH_PD
+Text Notes 6400 4550 3    50   ~ 0
+RESET
+Text Notes 6500 4550 3    50   ~ 0
+VCC
+Text Label 7050 1950 0    50   ~ 0
+GND
+Text Label 4800 3750 0    50   ~ 0
+FLASH
+Text Label 5450 5050 0    50   ~ 0
+RESET
+Text Label 5750 3650 0    50   ~ 0
+PC_TO_ESP
+Text Label 4850 4700 0    50   ~ 0
+ESP_TO_PC
 $EndSCHEMATC
